Commit message: Changed parent link of camera_link

File: urdf/robotr_description.urdf (robot description, URDF)
Before this commit: robot robotr_description, 26 links, 25 joints
Joints:
- joint kinect_camera_joint: parent base_link -> kinect

Commit message: Updated

File: urdf/robotr_description.urdf (robot description, URDF)
Before this commit: robot robotr_description, 26 links, 25 joints
Links:
- added link imu_link
Joints:
- added joint imu_joint: type fixed, parent upper_plate, child imu_link, origin xyz=0 0.04 0 rpy=0 0 0, axis 0 0 0
